File: Hardware/kicad/PUEiE_pcb/3_3V_Regulator.kicad_sch (KiCad schematic)
At the start: 18 parts, among them SW2 SW_DPDT_x2, U1 AMS1117-3.3, U5 TPS563240DDC

Commit message: Vbat
Parts:
- added C11: 100n, Capacitor_SMD:C_0805_2012Metric, symbol Device:C
- added D3: 3.3V, Diode_SMD:D_SOD-323, symbol Device:D_Schottky
- added R5: 40k, Resistor_SMD:R_0805_2012Metric, symbol Device:R
- added R6: 5.1 k, Resistor_SMD:R_0805_2012Metric, symbol Device:R
- added R8: 10k, Resistor_SMD:R_0805_2012Metric, symbol Device:R
- renumbered C12 to C1, C8 to C2, C9 to C3, C11 to C4, C13 to C5, C14 to C6, C15 to C7, C1 to C8, C2 to C9, D3 to D2, F2 to F1, L2 to L1, R5 to R1, R6 to R2, SW2 to SW1, U5 to U1, U1 to U5
Connections:
- net GND: now also C11.2, D3.2 (A), R8.2
- net +Vbat_fuse: now reaches C2.1, C3.1, C4.1, F1.2, U1.3 (VIN), U1.5 (EN)
- net +Vbat_fuse: now also R5.1
- new net: R5.2, R6.1, R8.1
- new net Vbat_adc: C11.1, D3.1 (K), R6.2
Other:
- note added: "+3.3V USB Regulator"
- note added: "Vbat adc"
- note added: "Vbat max 15V Vbat_adc max 3V f(-3dB) = 310 Hz"
- moved on the sheet: C1, C2, C3, C4, C5, C6, C7, C8, C9, D2, F1, JP2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
