File: Hardware/kicad/PUEiE_pcb/3_3V_Regulator.kicad_sch (KiCad schematic)
At the start: 25 parts, among them SW201 SW_DPDT_x2, U201 TPS563240DDC, U202 AMS1117-3.3

Commit message: All Schematics
Parts:
- removed SW201: SW_DPDT_x2, Button_Switch_THT:SW_E-Switch_EG1224_SPDT_Angled, symbol Switch:SW_DPDT_x2
- added SW201: SW_Nidec_CAS-120A1, Button_Switch_THT:SW_Slide-03_Wuerth-WS-SLTV_10x2.5x6.4_P2.54mm, symbol Switch:SW_Nidec_CAS-120A1
- added TP201, TP202, TP203: TestPoint, TestPoint:TestPoint_Pad_D2.0mm, symbol Connector:TestPoint
- C201: value 100nF -> 100n; Distributor (none) -> https://jlcpcb.com/partdetail/TaiyoYuden-EMK107B7104KAT/C38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; MFR Part (none) -> EMK107B7104KA-T; Manufacturer (none) -> Taiyo Yuden
- C202, C203: Distributor (none) -> https://jlcpcb.com/partdetail/367931-GRM21BR61E106MA73L/C39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; MFR Part (none) -> GRM21BR61E106MA73L; Manufacturer (none) -> Murata Electronics
- C204, C210: Distributor (none) -> https://jlcpcb.com/partdetail/28983-CL21B104KCFNNNE/C28233; MFR Part (none) -> CL21B104KCFNNNE; Manufacturer (none) -> Samsung Electro-Mechanics
- C205, C206, C207, C208, C209: Distributor (none) -> https://jlcpcb.com/partdetail/MurataElectronics-GRM188R60J2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; MFR Part (none) -> GRM188R60J226MEA0D; Manufacturer (none) -> Murata Electronics
- D201: footprint (none) -> Diode_SMD:D_SMA; Distributor (none) -> https://jlcpcb.com/partdetail/MDD_Microdiode_Semiconductor-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; MFR Part (none) -> SS34; Manufacturer (none) -> MDD(Microdiode Semiconductor)
- D202: Distributor (none) -> https://jlcpcb.com/partdetail/DiodesIncorporated-MMSZ5226BS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; Link 1 https://jlcpcb.com/partdetail/DiodesIncorporated-MMSZ5226BS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 -> (none); MFR Part (none) -> MMSZ5226BS-7-F; Manufacturer (none) -> Diodes Incorporated
- D203: Distributor (none) -> https://jlcpcb.com/partdetail/85425-NCD0805R1/C84256; MFR Part (none) -> NCD0805R1; Manufacturer (none) -> Foshan NationStar Optoelectronics
- F201: value 600mA -> 2A; footprint (none) -> Fuse:Fuseholder_Clip-5x20mm_Littelfuse_111_Inline_P20.00x5.00mm_D1.05mm_Horizontal; Distributor (none) -> https://jlcpcb.com/partdetail/XuchengElec-5x20/C3130; MFR Part (none) -> 5x20 环保 保险管夹/座; Manufacturer (none) -> Xucheng Elec
- JP201: footprint (none) -> Connector_PinHeader_2.54mm:PinHeader_1x03_P2.54mm_Vertical
- L201: Distributor (none) -> https://jlcpcb.com/partdetail/Sumida-104CDMCCDS1R5MC/C516064; MFR Part (none) -> 104CDMCCDS-1R5MC; Manufacturer (none) -> Sumida
- R201: footprint Resistor_SMD:R_0402_1005Metric -> Resistor_SMD:R_0805_2012Metric; Distributor (none) -> https://jlcpcb.com/partdetail/18389-0805W8F4532T5E/C17701; MFR Part (none) -> 0805W8F4532T5E; Manufacturer (none) -> UNI-ROYAL(Uniroyal Elec)
- R202: footprint Resistor_SMD:R_0201_0603Metric -> Resistor_SMD:R_0805_2012Metric; Distributor (none) -> https://jlcpcb.com/partdetail/18102-0805W8F1002T5E/C17414; MFR Part (none) -> 0805W8F1002T5E; Manufacturer (none) -> UNI-ROYAL(Uniroyal Elec)
- R203: Distributor (none) -> https://jlcpcb.com/partdetail/TEConnectivity-RH73H2A40MKTN/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; MFR Part (none) -> RH73H2A40MKTN; Manufacturer (none) -> TE Connectivity
- R204: Distributor (none) -> https://jlcpcb.com/partdetail/28584-0805W8F5101T5E/C27834; MFR Part (none) -> 0805W8F5101T5E; Manufacturer (none) -> UNI-ROYAL(Uniroyal Elec)
- R205: Distributor (none) -> https://jlcpcb.com/partdetail/26851-0805W8F1005T5E/C26108; MFR Part (none) -> 0805W8F1005T5E; Manufacturer (none) -> UNI-ROYAL(Uniroyal Elec)
- R206: Distributor (none) -> https://jlcpcb.com/partdetail/18245-0805W8F2200T5E/C17557; MFR Part (none) -> 0805W8F2200T5E; Manufacturer (none) -> UNI-ROYAL(Uniroyal Elec)
- U201: Distributor (none) -> https://jlcpcb.com/partdetail/TexasInstruments-TPS563240DDC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; Link 1 https://jlcpcb.com/partdetail/TexasInstruments-TPS563240DDC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 -> (none); MFR Part (none) -> TPS563240DDCR; Manufacturer (none) -> Texas Instruments
- U202: Distributor (none) -> https://jlcpcb.com/partdetail/Advanced_MonolithicSystems-AM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; Link 1 https://jlcpcb.com/partdetail/Advanced_MonolithicSystems-AM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 -> (none); MFR Part (none) -> AMS1117-3.3; Manufacturer (none) -> Advanced Monolithic Systems
Connections:
- net +3V3USB: now also TP201.1
- net Vbat+: now also SW201.2 (B)
- net Vbat_adc: now also TP203.1
- net Vbat_adc_in: now reaches R203.2, R204.1, R205.1
- net SBD_A: now reaches D201.2 (A)
- net SBD_A: now also SW201.3 (A)
- net at C205.1, C206.1, C207.1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: now also TP202.1
- net +3.3V_K: now reaches D203.1 (K), R206.1
- net SBD_K: now reaches D201.1 (K), F201.1
Other:
- note added: "10.5V - 15.0V"
- moved on the sheet: C208, C209, D201, D203, R206

Commit message: Board Setup
Parts:
- renumbered C210 to C208, C208 to C209, C209 to C210
Changed lines of the file:
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@@
 	)
 	(junction
+		(at 247.65 55.88)
+		(diameter 0)
+		(color 0 0 0 0)
+	)
+	(junction
 		(at 223.52 102.87)
 		(diameter 0)
@@
 	(wire
 		(pts
+			(xy 247.65 55.88) (xy 248.92 55.88)
+		)
+		(stroke
+			(width 0)
+			(type default)
+		)
+	)
+	(wire
+		(pts
 			(xy 167.64 29.21) (xy 167.64 26.67)
 		)
@@
 	(wire
 		(pts
-			(xy 245.11 55.88) (xy 248.92 55.88)
+			(xy 245.11 55.88) (xy 247.65 55.88)
 		)
 		(stroke
@@
 	)
 	(symbol
+		(lib_id "power:PWR_FLAG")
+		(at 247.65 55.88 0)
+		(unit 1)
+		(exclude_from_sim no)
+		(in_bom yes)
+		(on_board yes)
+		(dnp no)
+		(fields_autoplaced yes)
+		(property "Reference" "#FLG0205"
+			(at 247.65 53.975 0)
+			(effects
+				(font
+					(size 1.27 1.27)
+				)
+				(hide yes)
+			)
+		)
+		(property "Value" "PWR_FLAG"
+			(at 247.65 50.8 0)
+			(effects
+				(font
+					(size 1.27 1.27)
+				)
+				(hide yes)
+			)
+		)
+		(property "Footprint" ""
+			(at 247.65 55.88 0)
+			(effects
+				(font
+					(size 1.27 1.27)
+				)
+				(hide yes)
+			)
+		)
+		(property "Datasheet" "~"
+			(at 247.65 55.88 0)
+			(effects
+				(font
+					(size 1.27 1.27)
+				)
+				(hide yes)
+			)
+		)
+		(property "Description" "Special symbol for telling ERC where power comes from"
+			(at 247.65 55.88 0)
+			(effects
+				(font
+					(size 1.27 1.27)
+				)
+				(hide yes)
+			)
+		)
+		(pin "1"
+		)
+		(instances
+			(project "PUEiE_pcb"
+				(path "/064b0dc2-c3a5-4c74-8cbf-4fc3d8c84854/14f85070-237d-42f7-a449-5fde0a107bb8"
+					(reference "#FLG0205")
+					(unit 1)
+				)
+			)
+		)
+	)
+	(symbol
 		(lib_id "power:GND")
 		(at 212.09 160.02 0)
@@
 		(on_board yes)
 		(dnp no)
-		(property "Reference" "C208"
+		(property "Reference" "C209"
 			(at 197.866 105.41 0)
 			(effects
@@
 			(project "PUEiE_pcb"
 				(path "/064b0dc2-c3a5-4c74-8cbf-4fc3d8c84854/14f85070-237d-42f7-a449-5fde0a107bb8"
-					(reference "C208")
+					(reference "C209")
 					(unit 1)
 				)
@@
 		(on_board yes)
 		(dnp no)
-		(property "Reference" "C209"
+		(property "Reference" "C210"
 			(at 226.314 105.41 0)
 			(effects
@@
 			(project "PUEiE_pcb"
 				(path "/064b0dc2-c3a5-4c74-8cbf-4fc3d8c84854/14f85070-237d-42f7-a449-5fde0a107bb8"
-					(reference "C209")
+					(reference "C210")
 					(unit 1)
 				)
@@
 		(on_board yes)
 		(dnp no)
-		(property "Reference" "C210"
+		(property "Reference" "C208"
 			(at 80.01 110.49 0)
 			(effects
@@
 			(project "PUEiE_pcb"
 				(path "/064b0dc2-c3a5-4c74-8cbf-4fc3d8c84854/14f85070-237d-42f7-a449-5fde0a107bb8"
-					(reference "C210")
+					(reference "C208")
 					(unit 1)
 				)

Commit message: pcb placement
Parts:
- D203: value RED -> +3.3V
- U201: MFR Part TPS563240DDCR -> TPS563240DDCR
Connections:
- net +3.3Vbat: now reaches C205.1, C206.1, C207.1, JP201.3 (B), L201.2, R201.1, TP202.1
- net LDO_VFB: now reaches R201.2, R202.1, U201.4 (VFB)
- net LDO_SW: now reaches C201.1, L201.1, U201.2 (SW)
- net LDO_VBST: now reaches C201.2, U201.6 (VBST)
Changed lines of the file:
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@@
 		)
 	)
+	(label "+3.3Vbat"
+		(at 190.5 43.18 0)
+		(effects
+			(font
+				(size 0.5 0.5)
+			)
+			(justify left bottom)
+		)
+	)
+	(label "LDO_SW"
+		(at 163.83 26.67 0)
+		(effects
+			(font
+				(size 0.5 0.5)
+			)
+			(justify left bottom)
+		)
+	)
 	(label "SBD_K"
 		(at 87.63 43.18 0)
@@
 		)
 	)
+	(label "LDO_VFB"
+		(at 179.07 53.34 0)
+		(effects
+			(font
+				(size 0.5 0.5)
+			)
+			(justify left bottom)
+		)
+	)
 	(label "+3.3V_K"
 		(at 212.09 148.59 270)
@@
 		)
 	)
+	(label "LDO_VBST"
+		(at 162.56 45.72 0)
+		(effects
+			(font
+				(size 0.5 0.5)
+			)
+			(justify left bottom)
+		)
+	)
 	(hierarchical_label "Vbat+"
 		(shape output)
@@
 			)
 		)
-		(property "MFR Part" " TPS563240DDCR"
+		(property "MFR Part" "TPS563240DDCR"
 			(at 152.4 45.72 0)
 			(effects
@@
 			)
 		)
-		(property "Value" "RED"
+		(property "Value" "+3.3V"
 			(at 215.9 147.6374 90)
 			(effects
@@
 			)
 		)
-		(property "Description" "Light emitting diode"
+		(property "Description" "RED"
 			(at 212.09 144.78 0)
 			(effects

Commit message: PCB layout
Parts:
- SW201: footprint Button_Switch_THT:SW_Slide-03_Wuerth-WS-SLTV_10x2.5x6.4_P2.54mm -> Connector_PinHeader_2.54mm:PinHeader_1x03_P2.54mm_Vertical
- renumbered D203 to LD3V3
Changed lines of the file:
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@@
 			)
 		)
-		(property "Datasheet" "www.ti.com/lit/ds/symlink/tps563240.pdf"
+		(property "Datasheet" "https://www.ti.com/lit/ds/symlink/tps563240.pdf"
 			(at 152.4 45.72 0)
 			(effects
@@
 		(dnp no)
 		(fields_autoplaced yes)
-		(property "Reference" "D203"
-			(at 215.9 145.0974 90)
+		(property "Reference" "LD3V3"
+			(at 215.9 146.3674 90)
 			(effects
 				(font
@@
 				)
 				(justify right)
+				(hide yes)
 			)
 		)
@@
 			(project ""
 				(path "/064b0dc2-c3a5-4c74-8cbf-4fc3d8c84854/14f85070-237d-42f7-a449-5fde0a107bb8"
-					(reference "D203")
+					(reference "LD3V3")
 					(unit 1)
 				)
@@
 			)
 		)
-		(property "Footprint" "Button_Switch_THT:SW_Slide-03_Wuerth-WS-SLTV_10x2.5x6.4_P2.54mm"
+		(property "Footprint" "Connector_PinHeader_2.54mm:PinHeader_1x03_P2.54mm_Vertical"
 			(at 68.58 55.88 0)
 			(effects

Commit message: Final PCB design
Connections:
- net LDO_SW renamed SMPS_SW
- net LDO_VBST renamed SMPS_VBST
- net LDO_VFB renamed SMPS_VFB
Other:
- note added: "+3.3V SMPS Regulator"
- note removed: "+3.3V LDO Regulator"
Changed lines of the file:
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@@
 		)
 	)
-	(text "+3.3V LDO Regulator"
+	(text "+3.3V SMPS Regulator"
 		(exclude_from_sim no)
 		(at 147.32 18.542 0)
@@
 		)
 	)
-	(label "LDO_SW"
+	(label "SMPS_SW"
 		(at 163.83 26.67 0)
 		(effects
@@
 		)
 	)
-	(label "LDO_VFB"
+	(label "SMPS_VFB"
 		(at 179.07 53.34 0)
 		(effects
@@
 		)
 	)
-	(label "LDO_VBST"
+	(label "SMPS_VBST"
 		(at 162.56 45.72 0)
 		(effects
