File: Hardware/kicad/PUEiE_pcb/PUEiE_pcb.kicad_pcb (KiCad board)
At the start: 2 copper layers, 0 parts

Commit message: pcb placement
Parts:
- added C101: 4u7, Capacitor_SMD:C_0805_2012Metric, F.Cu at (139.4, 59.5)
- added C102: 100n, Capacitor_SMD:C_0805_2012Metric, F.Cu at (139.4, 61.6)
- added C103: 100p, Capacitor_SMD:C_0805_2012Metric, F.Cu at (151.6, 64.1)
- added C104: 100n, Capacitor_SMD:C_0805_2012Metric, F.Cu at (151.6, 62.0)
- added C105: 4u7, Capacitor_SMD:C_0805_2012Metric, F.Cu at (143.7, 29.0)
- added C106: 100n, Capacitor_SMD:C_0805_2012Metric, F.Cu at (135.9, 66.9)
- added C107: 100n, Capacitor_SMD:C_0805_2012Metric, F.Cu at (145.0, 73.5)
- added C108: 100n, Capacitor_SMD:C_0805_2012Metric, F.Cu at (136.4, 73.5)
- added C109: 100n, Capacitor_SMD:C_0805_2012Metric, F.Cu at (136.1, 63.1)
- added C110: 100n, Capacitor_SMD:C_0805_2012Metric, F.Cu at (151.6, 68.6)
- added C111: 100n, Capacitor_SMD:C_0805_2012Metric, F.Cu at (138.4, 73.5)
- added C112: 100n, Capacitor_SMD:C_0805_2012Metric, F.Cu at (145.0, 77.0)
- added C113: 100n, Capacitor_SMD:C_0805_2012Metric, F.Cu at (152.5, 49.6)
- added C114: 4u7, Capacitor_SMD:C_0805_2012Metric, F.Cu at (144.2, 61.6)
- added C115: 0p8, Capacitor_SMD:C_0402_1005Metric, F.Cu at (151.5, 66.3)
- added C116: 0p3, Capacitor_SMD:C_0402_1005Metric, F.Cu at (154.5, 66.3)
- added C117: 10p, Capacitor_SMD:C_0603_1608Metric, F.Cu at (141.8, 75.7)
- added C118: 10p, Capacitor_SMD:C_0603_1608Metric, F.Cu at (140.2, 75.7)
- added C119: 100n, Capacitor_SMD:C_0805_2012Metric, F.Cu at (148.8, 88.7)
- added C201: 100n, Capacitor_SMD:C_0603_1608Metric, F.Cu at (84.5, 23.7)
- added C202: 10u, Capacitor_SMD:C_0805_2012Metric, F.Cu at (75.0, 23.6)
- added C203: 10u, Capacitor_SMD:C_0805_2012Metric, F.Cu at (78.5, 23.6)
- added C204: 100n, Capacitor_SMD:C_0805_2012Metric, F.Cu at (82.0, 23.6)
- added C205: 22u, Capacitor_SMD:C_0603_1608Metric, F.Cu at (103.5, 23.8)
- added C206: 22u, Capacitor_SMD:C_0603_1608Metric, F.Cu at (106.0, 23.8)
- added C207: 22u, Capacitor_SMD:C_0603_1608Metric, F.Cu at (108.5, 23.8)
- added C208: 100n, Capacitor_SMD:C_0805_2012Metric, F.Cu at (127.3, 53.0)
- added C209: 22u, Capacitor_SMD:C_0603_1608Metric, F.Cu at (115.8, 52.9)
- added C210: 22u, Capacitor_SMD:C_0603_1608Metric, F.Cu at (117.8, 52.9)
- added C301: 100n, Capacitor_SMD:C_0805_2012Metric, F.Cu at (120.3, 90.0)
- added C302: 10u, Capacitor_SMD:C_0805_2012Metric, F.Cu at (129.3, 102.3)
- added C303: 47p, Capacitor_SMD:C_0805_2012Metric, F.Cu at (124.6, 103.2)
- added C304: 100n, Capacitor_SMD:C_0805_2012Metric, F.Cu at (152.8, 79.7)
- added C305: 1u, Capacitor_SMD:C_0805_2012Metric, F.Cu at (156.3, 79.7)
- added C306: 100n, Capacitor_SMD:C_0805_2012Metric, F.Cu at (149.3, 79.7)
- added C307: 100n, Capacitor_SMD:C_0805_2012Metric, F.Cu at (87.0, 97.8)
- added C308: 100u, Capacitor_SMD:CP_Elec_6.3x7.7, F.Cu at (85.6, 106.4)
- added C309: 100u, Capacitor_SMD:CP_Elec_6.3x7.7, F.Cu at (85.6, 114.5)
- added C310: 100n, Capacitor_SMD:C_0805_2012Metric, F.Cu at (87.0, 100.8)
- added C311: 100n, Capacitor_SMD:C_0805_2012Metric, F.Cu at (91.5, 91.7)
- added C312: 10u, Capacitor_SMD:C_0805_2012Metric, F.Cu at (91.5, 94.8)
- added C313: 10u, Capacitor_SMD:C_0805_2012Metric, F.Cu at (91.5, 97.8)
- added C314: 1u, Capacitor_SMD:C_0805_2012Metric, F.Cu at (91.5, 100.8)
- added C315: 100n, Capacitor_SMD:C_0805_2012Metric, F.Cu at (96.0, 91.7)
- added C316: 22n, Capacitor_SMD:C_0805_2012Metric, F.Cu at (96.0, 94.8)
- added C317: 2.2u, Capacitor_SMD:C_0805_2012Metric, F.Cu at (96.0, 97.8)
- added C318: 100n, Capacitor_SMD:C_0805_2012Metric, F.Cu at (158.5, 94.2)
- added D101: LD1, LED_SMD:LED_0805_2012Metric, F.Cu at (143.1, 45.1)
- added D201: D_Schottky, Diode_SMD:D_SMA, F.Cu at (50.5, 20.5)
- added D202: 3.3V, Diode_SMD:D_SOD-323, F.Cu at (129.4, 52.9)
- added D203: +3.3V, LED_SMD:LED_0805_2012Metric, F.Cu at (137.7, 45.1)
- added F201: 2A, Fuse:Fuseholder_Clip-5x20mm_Littelfuse_111_Inline_P20.00x5.00mm_D1.05mm_Horizontal, F.Cu at (48.0, 27.0)
- added J101: Screw_Terminal_01x02, TerminalBlock_Phoenix:TerminalBlock_Phoenix_PT-1,5-2-3.5-H_1x02_P3.50mm_Horizontal, F.Cu at (50.0, 33.0)
- added J102: USB_C_Receptacle_USB2.0_16P, Connector_USB:USB_C_Receptacle_GCT_USB4105-xx-A_16P_TopMnt_Horizontal, F.Cu at (100.1, 63.2)
- added J103: ST-LINKv2, Connector_PinHeader_1.27mm:PinHeader_2x05_P1.27mm_Vertical, F.Cu at (126.4, 64.2)
- added J104: Conn_IPEX, PUEiE_pcb_schematic_footprints:IPEX Male, F.Cu at (160.5, 65.9)
- added J301: Conn_IPEX, PUEiE_pcb_schematic_footprints:IPEX Male, F.Cu at (124.6, 107.7)
- added J302: SMD_JST_PHx04, Connector_JST:JST_XH_S4B-XH-A_1x04_P2.50mm_Horizontal, F.Cu at (63.6, 113.4)
- added J303: JST_PHx04, Connector_JST:JST_XH_S4B-XH-A_1x04_P2.50mm_Horizontal, F.Cu at (152.2, 98.3)
- added J304: Conn_01x03, Connector_JST:JST_XH_S3B-XH-A_1x03_P2.50mm_Horizontal, F.Cu at (49.6, 113.4)
- added JP201: Jumper_3_Bridged12, Connector_PinHeader_2.54mm:PinHeader_1x03_P2.54mm_Vertical, F.Cu at (115.5, 29.6)
- added JP301: SolderJumper_3_Bridged123, Jumper:SolderJumper-3_P2.0mm_Open_TrianglePad1.0x1.5mm, F.Cu at (117.0, 98.0)
- added JP302: SolderJumper_2_Open, Jumper:SolderJumper-2_P1.3mm_Open_TrianglePad1.0x1.5mm, F.Cu at (49.9, 91.2)
- added JP303: SolderJumper_2_Open, Jumper:SolderJumper-2_P1.3mm_Open_TrianglePad1.0x1.5mm, F.Cu at (49.9, 94.7)
- added JP304: SolderJumper_2_Open, Jumper:SolderJumper-2_P1.3mm_Open_TrianglePad1.0x1.5mm, F.Cu at (49.9, 98.2)
- added JP305: SolderJumper_2_Open, Jumper:SolderJumper-2_P1.3mm_Open_TrianglePad1.0x1.5mm, F.Cu at (49.9, 101.8)
- added JP306: SolderJumper_2_Open, Jumper:SolderJumper-2_P1.3mm_Open_TrianglePad1.0x1.5mm, F.Cu at (49.9, 105.3)
- added L101: 10u, Inductor_SMD:L_0603_1608Metric, F.Cu at (142.8, 59.6)
- added L102: 10n, Inductor_SMD:L_0402_1005Metric, F.Cu at (141.8, 61.6)
- added L103: 2n7, Inductor_SMD:L_0402_1005Metric, F.Cu at (153.0, 65.8)
- added L201: 1.5u, Inductor_SMD:L_Sunlord_MWSA1005S, F.Cu at (94.0, 23.5)
- added L301: 27n, Inductor_SMD:L_0402_1005Metric, F.Cu at (129.4, 104.2)
- added Q301: ZXMC4559DN8TA, Package_SO:SOP-8_3.76x4.96mm_P1.27mm, F.Cu at (137.5, 97.3)
- added R101: 0 ohm, Resistor_SMD:R_0805_2012Metric, F.Cu at (127.1, 61.8)
- added R102: 220R, Resistor_SMD:R_0805_2012Metric, F.Cu at (147.5, 49.6)
- added R103: 10k, Resistor_SMD:R_0805_2012Metric, F.Cu at (150.0, 49.6)
- added R104: 5.1k, Resistor_SMD:R_0805_2012Metric, F.Cu at (109.0, 60.4)
- added R105: 5.1k, Resistor_SMD:R_0805_2012Metric, F.Cu at (109.0, 66.3)
- added R106: 10k, Resistor_SMD:R_0805_2012Metric, F.Cu at (163.8, 88.7)
- added R107: 10k, Resistor_SMD:R_0805_2012Metric, F.Cu at (148.8, 85.7)
- added R108: 10k, Resistor_SMD:R_0805_2012Metric, F.Cu at (163.8, 85.7)
- added R109: 220R, Resistor_SMD:R_0805_2012Metric, F.Cu at (143.1, 48.6)
- added R201: 45.3k, Resistor_SMD:R_0805_2012Metric, F.Cu at (86.5, 34.1)
- added R202: 10k, Resistor_SMD:R_0805_2012Metric, F.Cu at (83.0, 34.1)
- added R203: 40M, Resistor_SMD:R_0805_2012Metric, F.Cu at (121.2, 53.0)
- added R204: 5.1k, Resistor_SMD:R_0805_2012Metric, F.Cu at (125.2, 53.0)
- added R205: 10M, Resistor_SMD:R_0805_2012Metric, F.Cu at (123.2, 53.0)
- added R206: 220R, Resistor_SMD:R_0805_2012Metric, F.Cu at (137.8, 48.6)
- added R301: 10R, Resistor_SMD:R_0603_1608Metric, F.Cu at (132.8, 105.1)
- added R302: 100k, Resistor_SMD:R_0603_1608Metric, F.Cu at (138.3, 92.1)
- added R303: 10k, Resistor_SMD:R_0805_2012Metric, F.Cu at (120.3, 96.5)
- added R304: 10k, Resistor_SMD:R_0805_2012Metric, F.Cu at (120.3, 100.0)
- added R305: 10k, Resistor_SMD:R_0805_2012Metric, F.Cu at (120.3, 93.0)
- added R306: 10k, Resistor_SMD:R_0805_2012Metric, F.Cu at (45.5, 99.7)
- added R307: 10k, Resistor_SMD:R_0805_2012Metric, F.Cu at (45.5, 102.7)
- added R308: 150m, Resistor_SMD:R_1206_3216Metric, F.Cu at (101.0, 91.9)
- added R309: 150m, Resistor_SMD:R_1206_3216Metric, F.Cu at (101.0, 95.2)
- added R310: 10k, Resistor_SMD:R_0805_2012Metric, F.Cu at (159.8, 79.8)
- added SW101: SW_Push, PUEiE_pcb_schematic_footprints:SW_2pin_5.5x2.0mm, F.Cu at (150.0, 45.6)
- added SW201: SW_Nidec_CAS-120A1, Button_Switch_THT:SW_Slide-03_Wuerth-WS-SLTV_10x2.5x6.4_P2.54mm, F.Cu at (52.0, 16.5)
- added TP201: TestPoint, TestPoint:TestPoint_Pad_D2.0mm, F.Cu at (116.9, 49.5)
- added TP202: TestPoint, TestPoint:TestPoint_Pad_D2.0mm, F.Cu at (106.0, 28.5)
- added TP203: TestPoint, TestPoint:TestPoint_Pad_D2.0mm, F.Cu at (132.5, 51.6)
- added TP301: TestPoint, TestPoint:TestPoint_Pad_D2.0mm, F.Cu at (54.1, 91.4)
- added TP302: TestPoint, TestPoint:TestPoint_Pad_D2.0mm, F.Cu at (54.1, 95.5)
- added TP303: TestPoint, TestPoint:TestPoint_Pad_D2.0mm, F.Cu at (54.1, 99.5)
- added TP304: TestPoint, TestPoint:TestPoint_Pad_D2.0mm, F.Cu at (54.1, 103.5)
- added U101: STM32WB55CGU6, Package_DFN_QFN:QFN-48-1EP_7x7mm_P0.5mm_EP5.6x5.6mm_ThermalVias, F.Cu at (143.3, 67.1)
- added U102: DLF162500LT-5028A1, PUEiE_pcb_schematic_footprints:DLF162500LT-5028A1, F.Cu at (156.5, 65.9)
- added U103: USBLC6-2SC6, Package_TO_SOT_SMD:SOT-23-6, F.Cu at (109.0, 63.5)
- added U104: W25Q128JVSIQ, Package_SO:SOIC-8_5.3x5.3mm_P1.27mm, F.Cu at (156.3, 87.2)
- added U201: TPS563240DDC, Package_TO_SOT_SMD:SOT-23-6, F.Cu at (84.4, 27.9)
- added U202: AMS1117-3.3, Package_TO_SOT_SMD:SOT-223-3_TabPin2, F.Cu at (110.8, 53.2)
- added U301: MAX-M10S-00B, RF_GPS:ublox_MAX, F.Cu at (127.8, 95.1)
- added U302: NC7WZ07P6X, Package_TO_SOT_SMD:SOT-363_SC-70-6, F.Cu at (132.8, 102.8)
- added U303: LIS3MDL, Package_LGA:LGA-12_2x2mm_P0.5mm, F.Cu at (155.3, 75.5)
- added U304: TMC2208-LA, Package_DFN_QFN:QFN-28-1EP_5x5mm_P0.5mm_EP3.75x3.75mm_ThermalVias, F.Cu at (66.7, 100.2)
- added Y101: 32MHz, Crystal:Crystal_SMD_2016-4Pin_2.0x1.6mm, F.Cu at (148.2, 60.8)
- added Y102: 32kHz768, Crystal:Crystal_SMD_2012-2Pin_2.0x1.2mm, F.Cu at (141.0, 73.0)
Routing:
- net +3V3: track 0.00 -> 43.0 mm
- net /Interfaces/GPS_VCC_RF: track 0.00 -> 5.53 mm
- net /HSE_IN: track 0.00 -> 4.50 mm
- net /MEM_~{HOLD}: track 0.00 -> 4.41 mm
- net /HSE_OUT: track 0.00 -> 4.37 mm
- net /MEM_~{WP}: track 0.00 -> 3.36 mm
- net /MEM_~{CS}: track 0.00 -> 3.17 mm
- net /USBD-: track 0.00 -> 2.48 mm
- net /USBD+: track 0.00 -> 2.44 mm
- net /VLXSMPS: track 0.00 -> 1.68 mm
- net (no net): track 0.00 -> 0.50 mm

Commit message: PCB layout
Parts:
- removed the C311 at (91.5, 91.7)
- removed the C313 at (91.5, 97.8)
- removed the C314 at (91.5, 100.8)
- removed JP305, JP306: SolderJumper_2_Open, Jumper:SolderJumper-2_P1.3mm_Open_TrianglePad1.0x1.5mm
- removed R101: 0 ohm, Resistor_SMD:R_0805_2012Metric
- removed TP303, TP304: TestPoint, TestPoint:TestPoint_Pad_D2.0mm
- added C312: 10u, Capacitor_SMD:C_1206_3216Metric, F.Cu at (110.3, 101.9)
- added FID1: Fiducial, Fiducial:Fiducial_1mm_Mask2mm, F.Cu at (105.2, 78.1)
- added FID2: Fiducial, Fiducial:Fiducial_1mm_Mask2mm, F.Cu at (139.0, 78.0)
- added FID3: Fiducial, Fiducial:Fiducial_1mm_Mask2mm, F.Cu at (139.0, 170.0)
- added FID4: Fiducial, Fiducial:Fiducial_1mm_Mask2mm, F.Cu at (105.2, 170.1)
- added FL301: SAW_GNSS, Filter:Filter_1109-5_1.1x0.9mm, F.Cu at (130.2, 161.3)
- added H1: MountingHole_Pad, MountingHole:MountingHole_3.2mm_M3_Pad, F.Cu at (100.2, 80.1)
- added H2: MountingHole_Pad, MountingHole:MountingHole_3.2mm_M3_Pad, F.Cu at (144.0, 80.0)
- added H3: MountingHole_Pad, MountingHole:MountingHole_3.2mm_M3_Pad, F.Cu at (144.0, 168.0)
- added H4: MountingHole_Pad, MountingHole:MountingHole_3.2mm_M3_Pad, F.Cu at (100.2, 168.1)
- C311: renamed from C312; footprint Capacitor_SMD:C_0805_2012Metric -> Capacitor_SMD:C_1206_3216Metric
- J304: value Conn_01x03 -> JST_PHx04; footprint Connector_JST:JST_XH_S3B-XH-A_1x03_P2.50mm_Horizontal -> Connector_JST:JST_XH_S4B-XH-A_1x04_P2.50mm_Horizontal
- SW201: footprint Button_Switch_THT:SW_Slide-03_Wuerth-WS-SLTV_10x2.5x6.4_P2.54mm -> Connector_PinHeader_2.54mm:PinHeader_1x03_P2.54mm_Vertical
- moved SW101 127.0 mm to (111.0, 166.5)
- moved R103 116.1 mm to (112.4, 159.5), turned to -90 degrees
- moved R102 116.1 mm to (110.0, 159.5), turned to -90 degrees
- moved C113 116.1 mm to (114.9, 159.5), turned to -90 degrees
- moved C105 102.1 mm to (121.8, 128.7), turned to 90 degrees
- moved R109 100.6 mm to (109.6, 143.5), turned to -90 degrees
- moved LD1 99.5 mm to (109.6, 138.7), turned to 90 degrees
- moved R206 98.0 mm to (113.3, 143.5), turned to -90 degrees
- moved LD3V3 96.8 mm to (113.3, 138.7), turned to 90 degrees
- moved SW201 93.3 mm to (106.0, 92.5), turned to 180 degrees
- moved C201 85.6 mm to (125.9, 98.7), turned to 180 degrees
- moved C205 85.2 mm to (135.1, 102.9)
- moved F201 85.2 mm to (114.7, 80.0)
- moved C206 84.9 mm to (136.9, 102.9)
- moved C207 84.7 mm to (138.7, 102.9)
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- renumbered C315 to C313, C316 to C314, C317 to C315, C318 to C316, D101 to LD1, D203 to LD3V3
Connections:
- C303 pad 2: /Interfaces/RF_IN -> /Interfaces/RF_IN_SAW
- J101 pad 1: GND -> /+3.3V Regulator/Vbat+
- J101 pad 2: /+3.3V Regulator/Vbat+ -> GND
- J103 pad 4: /ST_linkv2_3V3 -> unconnected-(J103-Pin_4-Pad4)
- J103 pad 7: /ST_linkv2_3V3 -> unconnected-(J103-Pin_7-Pad7)
- J304 pad 3: GND -> +3V3
- JP303 pad 2: /Interfaces/SMD_MS1 -> /Interfaces/SMD_MS2
- U304 pad 10: /Interfaces/SMD_MS1 -> /Interfaces/SMD_MS2
- U304 pad 21: /Interfaces/SMD_OA2 -> /Interfaces/SMD_OA1
- U304 pad 24: /Interfaces/SMD_OA1 -> /Interfaces/SMD_OA2
Routing:
- net +3V3: track 43.0 -> 70.8 mm
- net /Interfaces/GPS_EXTINT: track 0.00 -> 26.7 mm
- net /Interfaces/RF_IN_C: track 0.00 -> 12.9 mm
- net /Interfaces/GPS_VCC_RF: track 5.53 -> 17.7 mm
- net /Interfaces/GPS_LNA_EN: track 0.00 -> 11.6 mm
- net /Interfaces/SMD_DIAG_TP: track 0.00 -> 11.6 mm
- net /Interfaces/GPS_PMOS_G: track 0.00 -> 9.45 mm
- net /Interfaces/SMD_INDEX_TP: track 0.00 -> 8.88 mm
- net /Interfaces/GPS_EXTINT_BUF: track 0.00 -> 7.32 mm
- net /NRST: track 0.00 -> 7.10 mm
- net /Interfaces/GPS_PMOS_D: track 0.00 -> 5.64 mm
- net /SMD_ENN: track 0.00 -> 5.36 mm
- net /Interfaces/SMD_5VOUT: track 0.00 -> 4.56 mm
- net /MEM_~{HOLD}: track 4.41 -> 0.00 mm
- net /VFBSMPS: track 0.00 -> 4.30 mm
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- added copper zone on B.Cu, net GND
Other:
- board outline added: 52 x 96.1 mm
- board text added: "GND"
- board text added: "Vbat"

Commit message: Final PCB layout
Parts:
- J103: footprint Connector_PinHeader_1.27mm:PinHeader_2x05_P1.27mm_Vertical -> Connector_PinHeader_2.54mm:PinHeader_2x05_P2.54mm_Vertical
- moved TP201 13.9 mm to (110.6, 86.5)
- moved C210 10.4 mm to (111.1, 97.7)
- moved J103 9.80 mm to (111.2, 135.9), turned to 180 degrees
- moved R109 8.37 mm to (102.3, 147.5)
- moved LD1 8.37 mm to (102.3, 142.8)
- moved C311 7.70 mm to (106.5, 121.0)
- moved C310 7.70 mm to (105.9, 118.8)
- moved R206 7.66 mm to (106.8, 147.5)
- moved LD3V3 7.66 mm to (106.8, 142.8)
- moved C209 7.63 mm to (107.2, 97.7)
- moved C119 7.39 mm to (110.9, 142.8)
- moved R106 7.39 mm to (110.9, 147.5)
- moved R107 7.39 mm to (119.0, 142.7)
- moved R108 7.39 mm to (119.0, 147.5), turned to -90 degrees
- moved U104 7.39 mm to (115.0, 145.1)
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Connections:
- J103 pad 10: SWCLK -> unconnected-(J103-Pin_10-Pad10)
- J103 pad 2: unconnected-(J103-Pin_2-Pad2) -> SWCLK
- J103 pad 3: GND -> unconnected-(J103-Pin_3-Pad3)
- J103 pad 4: unconnected-(J103-Pin_4-Pad4) -> SWDIO
- J103 pad 5: unconnected-(J103-Pin_5-Pad5) -> GND
- J103 pad 6: unconnected-(J103-Pin_6-Pad6) -> GND
- J103 pad 8: GND -> unconnected-(J103-Pin_8-Pad8)
- J103 pad 9: SWDIO -> unconnected-(J103-Pin_9-Pad9)
- U101 pad 14: /MAG_~{CS} -> /SPI_SCK
- U101 pad 15: /SPI_SCK -> /SPI_MISO
- U101 pad 16: /SPI_MISO -> /SPI_MOSI
- U101 pad 17: /SPI_MOSI -> /MAG_~{CS}
- U101 pad 36: /USER_LED_A -> unconnected-(U101-PA10-Pad36)
- U101 pad 42: /ADC_VBAT -> /SMD_DIR
- U101 pad 43: /MOTOR_PWM -> /SMD_STEP
- U101 pad 44: /MOTOR_DIR -> /SMD_ENN
- U101 pad 45: /SMD_DIR -> /MOTOR_DIR
- U101 pad 46: /SMD_STEP -> /MOTOR_PWM
- U101 pad 47: /SMD_ENN -> /USER_LED_A
- U101 pad 9: unconnected-(U101-PA0-Pad9) -> /ADC_VBAT
- U103 pad 4: /USB_D- -> /USB_D+
- U103 pad 6: /USB_D+ -> /USB_D-
Routing:
- net +3V3: track 70.8 -> 373.1 mm, vias 0 -> 15
- net +Vbat_fuse: track 0.00 -> 190.0 mm, vias 0 -> 8
- net GND: track 0.00 -> 113.8 mm, vias 0 -> 345
- net /ADC_VBAT: track 0.00 -> 82.9 mm, vias 0 -> 6
- net VUSB: track 0.00 -> 70.3 mm, vias 0 -> 2
- net /I2C_SDA: track 0.00 -> 52.2 mm
- net /I2C_SCL: track 0.00 -> 48.9 mm
- net /BOOT0: track 0.00 -> 46.3 mm, vias 0 -> 2
- net /SPI_MISO: track 0.00 -> 45.1 mm, vias 0 -> 4
- net /MAG_~{CS}: track 0.00 -> 45.1 mm, vias 0 -> 2
- net /SPI_MOSI: track 0.00 -> 43.4 mm, vias 0 -> 2
- net /SPI_SCK: track 0.00 -> 42.5 mm, vias 0 -> 2
- net /MEM_~{CS}: track 0.00 -> 39.3 mm, vias 0 -> 2
- net /SMD_DIR: track 0.00 -> 39.2 mm, vias 0 -> 2
- net /SMD_STEP: track 0.00 -> 38.2 mm, vias 0 -> 2
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- added copper zone on F.Cu, net +3V3
- added copper zone on F.Cu, net +Vbat_fuse
- added copper zone on F.Cu, net /+3.3V Regulator/+3.3Vbat
- added copper zone on F.Cu, net /+3.3V Regulator/LDO_SW
- added copper zone on F.Cu, net /VFBSMPS
- added copper zone on F.Cu, net GND
Other:
- board size 52 x 96.1 mm -> 50 x 95 mm

Commit message: Final PCB design
Parts:
- JP302, JP303, TP301, TP302: moved to B.Cu
- moved TP301 2.00 mm to (117.5, 111.3), turned to 0 degrees
- moved TP302 2.00 mm to (117.5, 108.3), turned to 180 degrees
- moved JP302 1.87 mm to (114.5, 112.0)
- moved JP303 1.84 mm to (114.5, 107.8)
- moved C315 1.40 mm to (112.5, 113.5)
- moved C313 0.40 mm to (110.5, 114.5)
- moved C109 0.31 mm to (118.2, 116.8)
Connections:
- net /+3.3V Regulator/LDO_SW renamed /+3.3V Regulator/SMPS_SW
- net /+3.3V Regulator/LDO_VBST renamed /+3.3V Regulator/SMPS_VBST
- net /+3.3V Regulator/LDO_VFB renamed /+3.3V Regulator/SMPS_VFB
Routing:
- net /Interfaces/SMD_DIAG_TP: track 13.5 -> 7.95 mm, vias 0 -> 1
- net /SMD_DIR: track 39.2 -> 33.8 mm
- net /SMD_STEP: track 38.2 -> 32.8 mm
- net +3V3: track 373.1 -> 368.5 mm
- net /USB_D-: track 25.4 -> 29.4 mm
- net /Interfaces/SMD_INDEX_TP: track 11.0 -> 8.07 mm, vias 0 -> 1
- net /Interfaces/SMD_MS2: track 3.00 -> 5.76 mm, vias 0 -> 1
- net /Interfaces/SMD_MS1: track 2.61 -> 4.51 mm, vias 0 -> 1
- net /Interfaces/SMD_5VOUT: track 4.56 -> 3.17 mm
- net GND: track 113.8 -> 113.4 mm, vias 345 -> 406
