File: Hardware/kicad/PUEiE_pcb/PUEiE_pcb.kicad_sch (KiCad schematic)
At the start: 36 parts, among them J101 Screw_Terminal_01x02, J102 USB_C_Receptacle_USB2.0_16P, J103 ST-LINKv2, J104 Conn_IPEX, SW101 SW_Push, U101 STM32WB55CGU6, U102 DLF162500LT-5028A1, U103 USBLC6-2SC6, Y101 32MHz, Y102 32kHz768

Commit message: Board Setup
Parts:
- removed J103: ST-LINKv2, Connector_PinHeader_1.27mm:PinHeader_2x05_P1.27mm_Vertical, symbol STLINK-V3MINIE:STLINK-V3MINIE
- added J103: ST-LINKv2, Connector_PinHeader_1.27mm:PinHeader_2x05_P1.27mm_Vertical, symbol Connector_Generic:Conn_02x05_Counter_Clockwise
- renumbered C113 to C112, C112 to C113
Connections:
- net GND: now also J103.3 (Pin_3), J103.8 (Pin_8)
- net NRST: now also J103.1 (Pin_1)
- net ST_linkv2_3V3: now also J103.4 (Pin_4), J103.7 (Pin_7)
- net SWCLK: now also J103.10 (Pin_10)
- net SWDIO: now also J103.9 (Pin_9)
- net USART_RX: now also U101.36 (PA10); no longer U101.18 (PA9)
- net USART_TX: now also U101.18 (PA9); no longer U101.36 (PA10)
Other:
- moved on the sheet: J101

Commit message: pcb placement
Parts:
- added C119: 100n, Capacitor_SMD:C_0805_2012Metric, symbol Device:C
- added D101: LD1, LED_SMD:LED_0805_2012Metric, symbol Device:LED
- added R106, R107, R108: 10k, Resistor_SMD:R_0805_2012Metric, symbol Device:R
- added R109: 220R, Resistor_SMD:R_0805_2012Metric, symbol Device:R
- added U104: W25Q128JVSIQ, Package_SO:SOIC-8_5.3x5.3mm_P1.27mm, symbol Memory_Flash:W25Q128JVS
- U101: footprint Package_DFN_QFN:QFN-48-1EP_7x7mm_P0.5mm_EP5.6x5.6mm -> Package_DFN_QFN:QFN-48-1EP_7x7mm_P0.5mm_EP5.6x5.6mm_ThermalVias
- U103: MFR Part USBLC6-2SC6 -> USBLC6-2SC6
Connections:
- net +3V3: now also C101.2, C102.2, C105.2, C106.2, C109.2, C119.1, R106.1, R107.2, R108.2, U104.8 (VCC); no longer C101.1, C102.1, C105.1, C106.1, C109.1
- net ADC_VBAT: now also U101.42 (PA15); no longer U101.9 (PA0)
- net GND: now also C101.1, C102.1, C105.1, C106.1, C109.1, C119.2, R109.2, U104.4 (GND); no longer C101.2, C102.2, C105.2, C106.2, C109.2
- net MAG_~{CS}: now also U101.14 (PA5); no longer U101.44 (PB4)
- net MOTOR_DIR: now also U101.44 (PB4); no longer U101.43 (PB3)
- net MOTOR_PWM: now also U101.43 (PB3); no longer U101.42 (PA15)
- net SMD_DIR: now also U101.45 (PB5); no longer U101.46 (PB6)
- net SMD_STEP: now also U101.46 (PB6); no longer U101.45 (PB5)
- net SPI_MISO: now also U101.16 (PA7), U104.2 (DO/IO_{1}); no longer U101.15 (PA6)
- net SPI_MOSI: now also U101.17 (PA8), U104.5 (DI/IO_{0}); no longer U101.16 (PA7)
- net SPI_SCK: now also U101.15 (PA6), U104.6 (CLK); no longer U101.10 (PA1)
- net USART_RX: now also U101.12 (PA3); no longer U101.36 (PA10)
- net USART_TX: now also U101.11 (PA2); no longer U101.18 (PA9)
- net VFBSMPS: now also L101.2; no longer L102.2
- net VLXSMPS: now also L102.1; no longer L101.1
- net VLXSMPS_L: now also L101.1, L102.2; no longer L101.2, L102.1
- net ~{GPS_RESET}: now also U101.10 (PA1); no longer U101.19 (PB2)
- net MEM_~{CS}: now reaches U101.13 (PA4)
- net MEM_~{CS}: now also R106.2, U104.1 (~{CS})
- new net MEM_~{HOLD}: R107.1, U104.7 (~{HOLD}/~{RESET}/IO_{3})
- new net MEM_~{WP}: R108.1, U104.3 (~{WP}/IO_{2})
- new net USER_LED_A: D101.2 (A), U101.36 (PA10)
- new net USER_LED_K: D101.1 (K), R109.1
- no-connect marks 13 -> 11
Other:
- note added: "NRST button user led"
- moved on the sheet: C105, L101, L102

Commit message: PCB layout
Parts:
- removed R101: 0 ohm, Resistor_SMD:R_0805_2012Metric, symbol Device:R
- added FID1, FID2, FID3, FID4: Fiducial, Fiducial:Fiducial_1mm_Mask2mm, symbol Mechanical:Fiducial
- added H1, H2, H3, H4: MountingHole_Pad, MountingHole:MountingHole_3.2mm_M3_Pad, symbol Mechanical:MountingHole_Pad
- renumbered D101 to LD1
Connections:
- net +3.3V Regulator/Vbat+: now also J101.1 (Pin_1); no longer J101.2 (Pin_2)
- net +3.3V Regulator/Vbat-: now also J101.2 (Pin_2); no longer J101.1 (Pin_1)
- net GND: now also H1.1, H2.1, H3.1, H4.1
- net ST_linkv2_3V3: no longer names the net of J103.4 (Pin_4)
- net ST_linkv2_3V3: no longer J103.7 (Pin_7)
- no-connect marks 11 -> 13
Other:
- moved on the sheet: C113, J101, R102, R103, SW101, Y102

Commit message: Final PCB layout
Parts:
- removed J103: ST-LINKv2, Connector_PinHeader_1.27mm:PinHeader_2x05_P1.27mm_Vertical, symbol Connector_Generic:Conn_02x05_Counter_Clockwise
- added J103: ST-LINKv2, Connector_PinHeader_2.54mm:PinHeader_2x05_P2.54mm_Vertical, symbol Connector_Generic:Conn_02x05_Odd_Even
Connections:
- net ADC_VBAT: now also U101.9 (PA0); no longer U101.42 (PA15)
- net GND: now also J103.5 (Pin_5), J103.6 (Pin_6)
- net MAG_~{CS}: now also U101.17 (PA8); no longer U101.14 (PA5)
- net MOTOR_DIR: now also U101.45 (PB5); no longer U101.44 (PB4)
- net MOTOR_PWM: now also U101.46 (PB6); no longer U101.43 (PB3)
- net NRST: now also J103.1 (Pin_1)
- net SMD_DIR: now also U101.42 (PA15); no longer U101.45 (PB5)
- net SMD_ENN: now also U101.44 (PB4); no longer U101.47 (PB7)
- net SMD_STEP: now also U101.43 (PB3); no longer U101.46 (PB6)
- net SPI_MISO: now also U101.15 (PA6); no longer U101.16 (PA7)
- net SPI_MOSI: now also U101.16 (PA7); no longer U101.17 (PA8)
- net SPI_SCK: now also U101.14 (PA5); no longer U101.15 (PA6)
- net SWCLK: now also J103.2 (Pin_2)
- net SWDIO: now also J103.4 (Pin_4)
- net USB_D+: now also U103.4 (I/O2); no longer U103.6 (I/O1)
- net USB_D-: now also U103.6 (I/O1); no longer U103.4 (I/O2)
- net USER_LED_A: now also U101.47 (PB7); no longer U101.36 (PA10)
Other:
- note added: "U303 - czy mozna pod ic przelotke TP - czy mozna na drugiej stronie"
- note removed: "NRST button user led"
- moved on the sheet: LD1, R109

Commit message: Final PCB design
Other:
- note added: "Fiducial Mounting holes"
- note added: "Flash memory"
- note removed: "U303 - czy mozna pod ic przelotke TP - czy mozna na drugiej stronie"
- moved on the sheet: C101, C102, C103, C104, C105, C106, C107, C108, C109, C110, C111, C112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
